File: leech.kicad_pcb (KiCad board)
At the start: 2 copper layers, 17.8 x 43.2 mm, 15 parts, among them CN1 WeActBoard_noswd, U1 ICE40UP5K-SG48ITR, U2 STMPS2151STR, U3 TPS73101DBV

Commit message: Set solder mask params to zero to fix warning
Other:
- rule pad_to_mask_clearance: 0.05 -> 0
Changed lines of the file:
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@@
     (pad_size 1.524 1.524)
     (pad_drill 0.762)
-    (pad_to_mask_clearance 0.05)
-    (solder_mask_min_width 0.15)
+    (pad_to_mask_clearance 0)
     (aux_axis_origin 0 0)
     (visible_elements FFFDFF7F)
