File: leech.kicad_pcb (KiCad board)
At the start: 2 copper layers, 17.8 x 43.2 mm, 15 parts, among them CN1 WeActBoard_noswd, U1 ICE40UP5K-SG48ITR, U2 STMPS2151STR, U3 TPS73101DBV

Commit message: Bump board version (v1.1)
Other:
- board text added: "leech v1.1"
- board text removed: "leech v1.0"
Changed lines of the file:
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@@
       (net 2 /PILL_3V3))
   )
-  (gr_text "leech\nv1.0" (at 33.274 63.754 90) (layer B.Cu)
+  (gr_text "leech\nv1.1" (at 33.274 63.754 90) (layer B.Cu)
     (effects (font (size 1.2 1.2) (thickness 0.2)) (justify mirror))
   )
